File: MotorController.sch (EAGLE design)
At the start: 20 parts, among them IC1 MC33035, IC2 MC33039

Commit message: Adding.
Parts:
- removed R10: 1k, resistor:R-EU_0204/2V
- added C3, C4, C5, C8: 0.1uF, rcl:C-EU025-025X050
- added C7: 1000uF/50V, rcl:CPOL-EUE7.5-16
- added D1, D2: 1N4148DO35-7, diode:1N4148DO35-7
- added D3: 1N5819, diode:1N4148DO35-7
- added D4: 1N5352A, diode:1N5333
- added INC: (no value), SparkFun:TAC_SWITCHPTH
- added JP1: (no value), jumper:JP1E
- added R12, R13: 1k, resistor:R-EU_0204/2V
- added R14, R15: 1.1k, resistor:R-EU_0204/2V
- added R16, R17, R18: 470, resistor:R-EU_0204/2V
- added R20: 10k, pot:TRIM_EU-CA6V
- added R21: 0.05/1W, resistor:R-EU_0204/2V
- added R3B: 1M, resistor:R-EU_0204/2V
- added S1, S2, S3, S4, S5: (no value), switch:M251
- added TP1, TP2: TPPAD1-13Y, testpad:TPPAD1-13Y
- R3: value 1M -> 100k
- R6: value 470 -> 1.1k
- R7: value 470 -> 1k 0.5W
- R8: value 470 -> 100
- R9: value 1k -> 33
Connections:
- removed net N$1: IC2.8, R1.2
- removed net N$11: R6.1
- removed net N$12: R5.1
- removed net N$13: R10.1
- removed net N$14: R8.1
- removed net N$15: R9.1
- removed net N$16: R7.1
- removed net N$17: IC1.19
- removed net N$18: IC1.20
- removed net N$19: IC1.21
- removed net N$2: C1.1, R1.1
- removed net N$6: Q2.S, Q4.S, Q6.S
- new net 60/120: IC1.22, JP1.1
- new net AB: D3.C, IC1.21, R16.1
- new net ADJ: IC2.8, R1.2, R20.E, SL1.7
- new net AT: IC1.2, R5.1
- new net BB: D2.C, IC1.20, R17.1
- new net BRAKE: IC1.23, S5.P
- new net BT: IC1.1, R12.1
- new net CB: D1.C, IC1.19, R18.1
- new net CSENS: C5.1, IC1.9, R8.1, R9.2
- new net CT: IC1.24, R13.1
- new net ERRAMP: IC1.11, R20.S
- new net ERRA_N: C3.1, IC1.12, R3.2, R4.1, S3.P
- new net ERROUT: C3.2, IC1.13, R4.2, S3.S
- new net FAULT: IC1.14
- new net FOUT: IC2.5, R3.1
- new net RCT: C1.1, IC2.6, R1.1
- new net VC: C4.1, D4.C, IC1.18, R7.1
- net GND: now also C4.2, C5.2, C7.-, C8.2, D1.A, D2.A, D3.A, D4.A, IC1.15, IC1.16, JP1.2, R20.A, R21.1, R9.1, S5.S
- net N$10: now also R18.2; no longer R6.2
- net N$3: now also R17.2; no longer R8.2
- net N$4: now also R16.2; no longer R7.2
- net N$5: now also R5.2, R6.1; no longer R9.2
- net N$7: now also R21.2, R8.2
- net N$8: now also R12.2, R15.1; no longer R10.2
- net N$9: now also R13.2, R14.1; no longer R5.2
- net VCC: now also C7.+, C8.1, IC1.17, Q2.S, Q4.S, Q6.S, R14.2, R15.2, R6.2, R7.2; no longer SL1.7
Other:
- note added: "Remove if motor = 120"
- note removed: "Change DIL packages for SOIC."
- moved on the sheet: C1, Q1, Q2, Q3, Q4, Q5, Q6, R1, R3, R4, R5, R6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
